File: hardware/kicad/rescue-beacon-robot.kicad_sch (KiCad schematic)
At the start: 20 parts, among them M1 RB35GM_Encoder, M2 RB35GM_Encoder, SW1 SW_DPST_x2, U1 YDLIDAR_X4_Pro, U2 SZH-EK366_5V_5A_BUCK, U3 RDK_X5, U4 Cytron_MDD10A, U5 DFPlayer_Mini, U6 SZH-EKBD-066, U7 BNO085, U8 PAM8403

Commit message: 회로도 PDF 및 스키매틱 업데이트 추가, KiCad 락/자동저장 파일 gitignore 처리
Co-Authored-By: Claude Sonnet 5 <noreply@anthropic.com>
Parts:
- removed C1: 1000µF, symbol Device:C_Polarized
- removed M1, M2: RB35GM_Encoder, symbol RB35GM_Encoder:RB35GM_Encoder
- removed R5: 4.7k, symbol Device:R
- removed U4: Cytron_MDD10A, symbol Cytron_MDD10A:Cytron_MDD10A
- added M1, M2: 42-775B, symbol Motor_42-775B_Encoder:Motor_42-775B_Encoder
- added U4, U9: MD20A, symbol MD20A:MD20A
Connections:
- net +3.3V: now also U7.1 (VIN)
- net +5V: now also M1.3 (ENC_VCC), M2.3 (ENC_VCC)
- net GND: now also M1.4 (ENC_GND), M2.4 (ENC_GND), U4.3 (GND), U4.7 (VB-), U9.3 (GND), U9.7 (VB-)
- net ENC_R_B: now reaches A2.11 (D8)
- net ENC_R_B: now also M2.6 (ENC_B)
- net ENC_L_A: now reaches A2.5 (D2)
- net ENC_L_A: now also M1.5 (ENC_A)
- net ENC_L_B: now reaches A2.8 (D5)
- net ENC_L_B: now also M1.6 (ENC_B)
- net ENC_R_A: now reaches A2.9 (D6)
- net ENC_R_A: now also M2.5 (ENC_A)
- net DIR1 renamed DIR_L
- net DIR_L: now also U4.2 (DIR)
- net DIR2 renamed DIR_R
- net DIR_R: now also U9.2 (DIR)
- net PWM1 renamed PWM_L
- net PWM_L: now also U4.1 (PWM)
- net PWM2 renamed PWM_R
- net PWM_R: now also U9.1 (PWM)
- new net: M2.1 (M+), U9.5 (MB)
- new net: M2.2 (M-), U9.4 (MA)
- new net: M1.1 (M+), U4.4 (MA)
- new net: M1.2 (M-), U4.5 (MB)
- new net +22.2V: U4.6 (VB+), U9.6 (VB+)
Other:
- moved on the sheet: A2, R1, R2, R3, R4

Commit message: 회로도 수정
Co-Authored-By: Claude Sonnet 5 <noreply@anthropic.com>
Parts:
- BT1: value 11.1V -> +22.2V
Connections:
- net +11.1V is gone; now on net +22.2V: SW1.2 (B), U2.1 (VIN+), U6.1 (VIN+)
Changed lines of the file:
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@@
 			)
 		)
-		(property "Value" "+11.1V"
-			(at 71.12 22.86 0)
-			(effects
-				(font
-					(size 1.27 1.27)
-				)
+		(property "Value" "+22.2V"
+			(at 73.66 26.6699 0)
+			(effects
+				(font
+					(size 1.27 1.27)
+				)
+				(justify left)
 			)
 		)
@@
 			)
 		)
-		(property "Value" "11.1V"
+		(property "Value" "+22.2V"
 			(at 37.4015 30.48 90)
 			(effects
